File: himax_integration_5.kicad_pcb (KiCad board)
At the start: 2 copper layers, 16.8 x 8.2 mm, 30 parts, among them J1 VBat, J2 GND Pad, J3 SWDCLK Pad, J4 SWDIO Pad, J5 RST Pad, J6 Antenna Pad, Q2 Q_NPN, U1 ICM-42688-P, U2 MAG_Switch, U3 ES2832AA2

Commit message: restructured with local libs
Parts:
- HM01B1: footprint camera_flexa:camerah -> HM01B0:camerah
- J1, J2, J3, J4, J5, J6: footprint Connector_Pin:ExternalPad_FP -> himax_custom:ExternalPad_FP
- Q2: footprint Package_TO_SOT_SMD:SOT-883_1 -> himax_custom:SOT-883_1
- REF**: footprint Resistor_SMD:0hm 0603 metric 0.30 mm spacing -> himax_custom:0hm 0603 metric 0.30 mm spacing
- U1: footprint camera_flexa:PQFN50P300X250X97-14N -> ICM-42688-P:PQFN50P300X250X97-14N
- U2: footprint kicad_fp_sch_vreg:RR122 -> RR122:RR122
- U3: footprint ES2832AA2 (1):XCVR_ES2832AA2 -> ES2832AA2:XCVR_ES2832AA2_NO_ANTENNA
Changed lines of the file:
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@@
 		)
 	)
-	(footprint "kicad_fp_sch_vreg:RR122"
+	(footprint "RR122:RR122"
 		(layer "F.Cu")
 		(at 176.625 87.475 90)
@@
 		(embedded_fonts no)
 	)
-	(footprint "camera_flexa:PQFN50P300X250X97-14N"
+	(footprint "ICM-42688-P:PQFN50P300X250X97-14N"
 		(layer "F.Cu")
 		(at 178.202 84.071 90)
@@
 			)
 		)
-		(attr smd dnp)
+		(attr smd)
 		(duplicate_pad_numbers_are_jumpers no)
 		(fp_poly
@@
 		(embedded_fonts no)
 	)
-	(footprint "Connector_Pin:ExternalPad_FP"
+	(footprint "himax_custom:ExternalPad_FP"
 		(layer "F.Cu")
 		(at 170.169 81.563)
@@
 		)
 	)
-	(footprint "Package_TO_SOT_SMD:SOT-883_1"
+	(footprint "himax_custom:SOT-883_1"
 		(layer "F.Cu")
 		(at 170.365 87.221 90)
@@
 		)
 	)
-	(footprint "Connector_Pin:ExternalPad_FP"
+	(footprint "himax_custom:ExternalPad_FP"
 		(layer "F.Cu")
 		(at 171.12 81.545)
@@
 		)
 	)
-	(footprint "Connector_Pin:ExternalPad_FP"
+	(footprint "himax_custom:ExternalPad_FP"
 		(layer "F.Cu")
 		(at 168.419 81.544)
@@
 		)
 	)
-	(footprint "camera_flexa:camerah"
+	(footprint "HM01B0:camerah"
 		(layer "F.Cu")
 		(at 166.773 84.473 90)
@@
 		)
 	)
-	(footprint "Connector_Pin:ExternalPad_FP"
+	(footprint "himax_custom:ExternalPad_FP"
 		(layer "F.Cu")
 		(at 173.973 81.544)
@@
 		(embedded_fonts no)
 	)
-	(footprint "Resistor_SMD:0hm 0603 metric 0.30 mm spacing"
+	(footprint "himax_custom:0hm 0603 metric 0.30 mm spacing"
 		(layer "F.Cu")
 		(at 178.594 86.23 180)
@@
 		)
 	)
-	(footprint "ES2832AA2 (1):XCVR_ES2832AA2"
+	(footprint "ES2832AA2:XCVR_ES2832AA2_NO_ANTENNA"
 		(layer "F.Cu")
 		(at 172.446 84.177)
@@
 		(embedded_fonts no)
 	)
-	(footprint "Connector_Pin:ExternalPad_FP"
+	(footprint "himax_custom:ExternalPad_FP"
 		(layer "F.Cu")
 		(at 174.712 88.842)
@@
 		(embedded_fonts no)
 	)
-	(footprint "Connector_Pin:ExternalPad_FP"
+	(footprint "himax_custom:ExternalPad_FP"
 		(layer "F.Cu")
 		(at 171.955 81.545)
